Commit message: added cam mount (broken)

File: hrvip/hrvip_bringup/urdf/a_bot.urdf.xacro (robot description, xacro)
@@ -1,112 +1,68 @@
 <?xml version="1.0"?>
 <robot xmlns:xacro="http://wiki.ros.org/xacro" name="a_bot">
-  <!-- robot name parameter -->
-  <xacro:arg name="name" default="a_bot"/>
-  <!-- import main macro -->
+  <!-- import macro -->
+  <xacro:include filename="$(find robotiq_description)/urdf/robotiq_2f_85_macro.urdf.xacro" />
   <xacro:include filename="$(find ur_description)/urdf/ur_macro.xacro"/>
-  <!-- possible 'ur_type' values: ur3, ur3e, ur5, ur5e, ur10, ur10e, ur16e, ur20, ur30 -->
-  <!-- the default value should raise an error in case this was called without defining the type -->
-  <xacro:arg name="ur_type" default="ur5e"/>
+  <xacro:include filename="$(find hrvip_bringup)/urdf/d415_mount_macro.xacro"/>
   <!-- parameters -->
   <xacro:arg name="tf_prefix" default="" />
-  <xacro:arg name="joint_limit_params" default="$(find ur_description)/config/$(arg ur_type)/joint_limits.yaml"/>
-  <xacro:arg name="kinematics_params" default="$(find hrvip_bringup)/config/a_bot_calibration.yaml"/>
-  <xacro:arg name="physical_params" default="$(find ur_description)/config/$(arg ur_type)/physical_parameters.yaml"/>
-  <xacro:arg name="visual_params" default="$(find ur_description)/config/$(arg ur_type)/visual_parameters.yaml"/>
-  <xacro:arg name="transmission_hw_interface" default=""/>
-  <xacro:arg name="safety_limits" default="false"/>
-  <xacro:arg name="safety_pos_margin" default="0.15"/>
-  <xacro:arg name="safety_k_position" default="20"/>
-  <!-- ros2_control related parameters -->
+  <xacro:arg name="robot_ip" default="0.0.0.0" />
+  <xacro:arg name="reverse_ip" default="0.0.0.0"/>
   <xacro:arg name="headless_mode" default="false" />
-  <xacro:arg name="robot_ip" default="0.0.0.0" />
-  <xacro:arg name="script_filename" default=""/>
-  <xacro:arg name="output_recipe_filename" default=""/>
-  <xacro:arg name="input_recipe_filename" default=""/>
-  <xacro:arg name="reverse_ip" default="0.0.0.0"/>
-  <xacro:arg name="script_command_port" default="50004"/>
-  <xacro:arg name="reverse_port" default="50001"/>
-  <xacro:arg name="script_sender_port" default="50002"/>
-  <xacro:arg name="trajectory_port" default="50003"/>
   <!--   tool communication related parameters-->
   <xacro:arg name="use_tool_communication" default="true" />
   <xacro:arg name="tool_voltage" default="24" />
-  <xacro:arg name="tool_parity" default="0" />
-  <xacro:arg name="tool_baud_rate" default="115200" />
-  <xacro:arg name="tool_stop_bits" default="1" />
-  <xacro:arg name="tool_rx_idle_chars" default="1.5" />
-  <xacro:arg name="tool_tx_idle_chars" default="3.5" />
   <xacro:arg name="tool_device_name" default="/tmp/ttyUR" />
   <xacro:arg name="tool_tcp_port" default="54321" />
-    <!-- Simulation parameters -->
+  <!-- Simulation parameters -->
   <xacro:arg name="use_fake_hardware" default="false" />
   <xacro:arg name="fake_sensor_commands" default="false" />
-  <xacro:arg name="sim_gazebo" default="false" />
-  <xacro:arg name="sim_ignition" default="false" />
-  <xacro:arg name="simulation_controllers" default="" />
   <!-- initial position for simulations (Fake Hardware, Gazebo, Ignition) -->
   <xacro:arg name="initial_positions_file" default="$(find ur_description)/config/initial_positions.yaml"/>
   <!-- convert to property to use substitution in function -->
   <xacro:property name="initial_positions_file" default="$(arg initial_positions_file)"/>
-  <!-- gripper args/params -->
-  <xacro:include filename="$(find robotiq_description)/urdf/robotiq_2f_85_macro.urdf.xacro" />
   <!-- create link fixed to the "world" -->
   <link name="world" />
   <!-- arm -->
   <xacro:ur_robot
-    name="$(arg name)"
+    name="ur5e"
     tf_prefix="$(arg tf_prefix)"
     parent="world"
-    joint_limits_parameters_file="$(arg joint_limit_params)"
-    kinematics_parameters_file="$(arg kinematics_params)"
-    physical_parameters_file="$(arg physical_params)"
-    visual_parameters_file="$(arg visual_params)"
-    transmission_hw_interface="$(arg transmission_hw_interface)"
-    safety_limits="$(arg safety_limits)"
-    safety_pos_margin="$(arg safety_pos_margin)"
-    safety_k_position="$(arg safety_k_position)"
+    joint_limits_parameters_file="$(find ur_description)/config/ur5e/joint_limits.yaml"
+    kinematics_parameters_file="$(find hrvip_bringup)/config/a_bot_calibration.yaml"
+    physical_parameters_file="$(find ur_description)/config/ur5e/physical_parameters.yaml"
+    visual_parameters_file="$(find ur_description)/config/ur5e/visual_parameters.yaml"
     use_fake_hardware="$(arg use_fake_hardware)"
     fake_sensor_commands="$(arg fake_sensor_commands)"
-    sim_gazebo="$(arg sim_gazebo)"
-    sim_ignition="$(arg sim_ignition)"
-    headless_mode="$(arg headless_mode)"
     initial_positions="${xacro.load_yaml(initial_positions_file)}"
     use_tool_communication="$(arg use_tool_communication)"
     tool_voltage="$(arg tool_voltage)"
-    tool_parity="$(arg tool_parity)"
-    tool_baud_rate="$(arg tool_baud_rate)"
-    tool_stop_bits="$(arg tool_stop_bits)"
-    tool_rx_idle_chars="$(arg tool_rx_idle_chars)"
-    tool_tx_idle_chars="$(arg tool_tx_idle_chars)"
     tool_device_name="$(arg tool_device_name)"
     tool_tcp_port="$(arg tool_tcp_port)"
     robot_ip="$(arg robot_ip)"
-    script_filename="$(arg script_filename)"
-    output_recipe_filename="$(arg output_recipe_filename)"
-    input_recipe_filename="$(arg input_recipe_filename)"
     reverse_ip="$(arg reverse_ip)"
-    script_command_port="$(arg script_command_port)"
-    reverse_port="$(arg reverse_port)"
-    script_sender_port="$(arg script_sender_port)"
-    trajectory_port="$(arg trajectory_port)"
-    >
+    headless_mode="$(arg headless_mode)"
+    generate_ros2_control_tag="true"
+  >
     <origin xyz="0 0 0" rpy="0 0 0" />          <!-- position robot in the world -->
   </xacro:ur_robot>
+  <xacro:d415_mount
+    prefix="$(arg tf_prefix)"
+    parent="$(arg tf_prefix)wrist_3_link"
+    include_camera="true"
+  >
+    <origin xyz="0 0 0" rpy="0 0 0" />
+  </xacro:d415_mount>
   <xacro:robotiq_gripper
     name="RobotiqGripperHardwareInterface"
     com_port="$(arg tool_device_name)"
     prefix="$(arg tf_prefix)"
-    parent="$(arg tf_prefix)wrist_3_link"
+    parent="$(arg tf_prefix)d415_mount_attach_link"
     include_ros2_control="true"
     use_fake_hardware="$(arg use_fake_hardware)"
     fake_sensor_commands="$(arg fake_sensor_commands)"
+    grasp_link_offset="0.15"
   >
     <origin xyz="0 0 0" rpy="0 0 0" />
   </xacro:robotiq_gripper>
-  <link name="$(arg tf_prefix)grasp_link" />
-  <joint name="$(arg tf_prefix)grasp_joint" type="fixed">
-    <parent link="$(arg tf_prefix)robotiq_85_base_link" />
-    <child link="$(arg tf_prefix)grasp_link" />
-    <origin xyz="0.0 0.0 0.15" rpy="0 0 0" />
-  </joint>
 </robot>
